File: test01.kicad_pcb (KiCad board)
At the start: 2 copper layers, 668 x 398 mm, 2 parts, among them J1 Conn_01x01_Pin, J2 Conn_01x01_Pin

Commit message: save przed lengthmatchingiem lewa strona
Routing:
- net /TRACE: track 17580.8 -> 9153.0 mm

Commit message: test bofe matching
Routing:
- net /TRACE: track 9153.0 -> 8744.5 mm

Commit message: test nowy layout przed matchingime
Routing:
- net /TRACE: track 8744.5 -> 8719.6 mm

Commit message: test nowy #232
Routing:
- net /TRACE: track 8719.6 -> 8424.1 mm

Commit message: routing z kompa K
Routing:
- net /TRACE: track 8424.1 -> 44968.8 mm

Commit message: wip
Routing:
- net /TRACE: track 44968.8 -> 44071.3 mm
