File: test01.kicad_pcb (KiCad board)
At the start: 2 copper layers, 668 x 398 mm, 155 parts, among them J1 Conn_01x01_Pin, J2 Conn_01x01_Pin

Commit message: do ogarnięcia poprawione rzędy i sprawdzić odległości między ścieżkami
Routing:
- net /TRACE: track 67453.9 -> 67538.9 mm

Commit message: .
Parts:
- removed the ? at (529.5, 424.0)
- removed the ? at (530.2, 389.7)
- removed the ? at (367.1, 380.3)
- removed the ? at (366.8, 380.6)
- added ?: , , F.Cu at (367.5, 470.9)
Routing:
- net /TRACE: track 67538.9 -> 67467.9 mm
